Commit message: added message and changed urdf file advanded user guide gives 60 degrees transform for link 4 and 5

File: jaco_description/urdf/jaco_arm.urdf.xacro (robot description, xacro)
@@ -45,9 +45,9 @@
   <xacro:property name="joint_5_axis_xyz" value="0 0 1" />
   <xacro:property name="joint_5_origin_xyz" value="0.0343 0 -0.06588" />
-  <xacro:property name="joint_5_origin_rpy" value="0 ${M_PI/180*55} ${M_PI}" />
+  <xacro:property name="joint_5_origin_rpy" value="0 ${M_PI/180*60} ${M_PI}" />
   <xacro:property name="joint_6" value="jaco_joint_6" />
   <xacro:property name="joint_6_axis_xyz" value="0 0 1" />
   <xacro:property name="joint_6_origin_xyz" value="0.0343 0 -0.06588" />
-  <xacro:property name="joint_6_origin_rpy" value="0 ${M_PI/180*55} ${M_PI}" />
+  <xacro:property name="joint_6_origin_rpy" value="0 ${M_PI/180*60} ${M_PI}" />
   <xacro:property name="joint_finger_1" value="jaco_joint_finger_1" />
   <xacro:property name="joint_finger_1_axis_xyz" value="0 0 1" />

Commit message: model change joint 5 and 6 transform: rotate 60 degrees instead of 55. specified in handbook

File: jaco_description/urdf/jaco_arm.urdf.xacro (robot description, xacro)
@@ -45,9 +45,9 @@
   <xacro:property name="joint_5_axis_xyz" value="0 0 1" />
   <xacro:property name="joint_5_origin_xyz" value="0.0343 0 -0.06588" />
-  <xacro:property name="joint_5_origin_rpy" value="0 ${M_PI/180*60} ${M_PI}" />
+  <xacro:property name="joint_5_origin_rpy" value="0 ${M_PI/180*60} ${M_PI}" /> <!-- maybe 55 degrees, Advanded user guide specifys 60 ...-->
   <xacro:property name="joint_6" value="jaco_joint_6" />
   <xacro:property name="joint_6_axis_xyz" value="0 0 1" />
   <xacro:property name="joint_6_origin_xyz" value="0.0343 0 -0.06588" />
-  <xacro:property name="joint_6_origin_rpy" value="0 ${M_PI/180*60} ${M_PI}" />
+  <xacro:property name="joint_6_origin_rpy" value="0 ${M_PI/180*60} ${M_PI}" /> <!-- maybe 55 degrees, Advanded user guide specifys 60 ...-->
   <xacro:property name="joint_finger_1" value="jaco_joint_finger_1" />
   <xacro:property name="joint_finger_1_axis_xyz" value="0 0 1" />

Commit message: fixed acc frames; dynamic reconf priority ques

File: jaco_description/urdf/jaco_arm.urdf.xacro (robot description, xacro)
@@ -26,5 +26,5 @@
 	<xacro:property name="joint_base" value="jaco_joint_base" />
 	<xacro:property name="joint_base_axis_xyz" value="0 0 0" />
-	<xacro:property name="joint_1" value="jaco_joint_1" />
+  <xacro:property name="joint_1" value="jaco_joint_1" />
   <xacro:property name="joint_1_axis_xyz" value="0 0 1" />
   <xacro:property name="joint_1_origin_xyz" value="0 0 0.1535" />

Commit message: jaco2 kinematics and dynamics forward kinematics and inverse dynamics

File: jaco_description/urdf/jaco_arm.urdf.xacro (robot description, xacro)
@@ -91,5 +91,5 @@
                 <mass value="1"/>
                 <inertia ixx="0.1" ixy="0" ixz="0" iyy="0.1" iyz="0" izz="0.1"/>
-                <origin/>
+                <origin xyz="0.01 0.01 0.01" rpy="0 0 0"/>
             </inertial>
 			<visual>

Commit message: dynamic parameters avavible in urdf; ik solver in jaco2_kin_dyn <-- to be tested

File: jaco_description/urdf/jaco_arm.urdf.xacro (robot description, xacro)
@@ -13,5 +13,5 @@
 	xmlns:physics="http://playerstage.sourceforge.net/gazebo/xmlschema/#physics"
 	xmlns:xacro="http://ros.org/wiki/xacro">
-  <xacro:property name="M_SCALE" value="0.0254" />
+    <xacro:property name="M_SCALE" value="0.0254" />
 	<xacro:property name="M_PI" value="3.1415926535897931" />
 	<xacro:property name="J_LIM" value="${2*M_PI}" />
@@ -86,10 +86,73 @@
   <xacro:property name="joint_finger_tip_3_lower_limit" value="0" />
   <xacro:property name="joint_finger_tip_3_upper_limit" value="${M_PI/180*40}" />
-	<xacro:macro name="jaco_link" params="link_name">
+  <xacro:property name="link_base_com_xyz" value="0 0 0" />
+  <xacro:property name="link_base_com_rpy" value="0 0 0" />
+  <xacro:property name="link_base_mass" value="0.1" />
+  <xacro:property name="link_base_Ixx" value="0.1" />
+  <xacro:property name="link_base_Ixy" value="0.0" />
+  <xacro:property name="link_base_Ixz" value="0.0" />
+  <xacro:property name="link_base_Iyy" value="0.1" />
+  <xacro:property name="link_base_Iyz" value="0.0" />
+  <xacro:property name="link_base_Izz" value="0.1" />
+  <xacro:property name="link_1_com_xyz" value="0 0 0" />
+  <xacro:property name="link_1_com_rpy" value="0 0 0" />
+  <xacro:property name="link_1_mass" value="0.1" />
+  <xacro:property name="link_1_Ixx" value="0.1" />
+  <xacro:property name="link_1_Ixy" value="0.0" />
+  <xacro:property name="link_1_Ixz" value="0.0" />
+  <xacro:property name="link_1_Iyy" value="0.1" />
+  <xacro:property name="link_1_Iyz" value="0.0" />
+  <xacro:property name="link_1_Izz" value="0.1" />
+  <xacro:property name="link_2_com_xyz" value="0 0 0" />
+  <xacro:property name="link_2_com_rpy" value="0 0 0" />
+  <xacro:property name="link_2_mass" value="0.1" />
+  <xacro:property name="link_2_Ixx" value="0.1" />
+  <xacro:property name="link_2_Ixy" value="0.0" />
+  <xacro:property name="link_2_Ixz" value="0.0" />
+  <xacro:property name="link_2_Iyy" value="0.1" />
+  <xacro:property name="link_2_Iyz" value="0.0" />
+  <xacro:property name="link_2_Izz" value="0.1" />
+  <xacro:property name="link_3_com_xyz" value="0 0 0" />
+  <xacro:property name="link_3_com_rpy" value="0 0 0" />
+  <xacro:property name="link_3_mass" value="0.1" />
+  <xacro:property name="link_3_Ixx" value="0.1" />
+  <xacro:property name="link_3_Ixy" value="0.0" />
+  <xacro:property name="link_3_Ixz" value="0.0" />
+  <xacro:property name="link_3_Iyy" value="0.1" />
+  <xacro:property name="link_3_Iyz" value="0.0" />
+  <xacro:property name="link_3_Izz" value="0.1" />
+  <xacro:property name="link_4_com_xyz" value="0 0 0" />
+  <xacro:property name="link_4_com_rpy" value="0 0 0" />
+  <xacro:property name="link_4_mass" value="0.1" />
+  <xacro:property name="link_4_Ixx" value="0.1" />
+  <xacro:property name="link_4_Ixy" value="0.0" />
+  <xacro:property name="link_4_Ixz" value="0.0" />
+  <xacro:property name="link_4_Iyy" value="0.1" />
+  <xacro:property name="link_4_Iyz" value="0.0" />
+  <xacro:property name="link_4_Izz" value="0.1" />
+  <xacro:property name="link_5_com_xyz" value="0 0 0" />
+  <xacro:property name="link_5_com_rpy" value="0 0 0" />
+  <xacro:property name="link_5_mass" value="0.1" />
+  <xacro:property name="link_5_Ixx" value="0.1" />
+  <xacro:property name="link_5_Ixy" value="0.0" />
+  <xacro:property name="link_5_Ixz" value="0.0" />
+  <xacro:property name="link_5_Iyy" value="0.1" />
+  <xacro:property name="link_5_Iyz" value="0.0" />
+  <xacro:property name="link_5_Izz" value="0.1" />
+  <xacro:property name="link_hand_com_xyz" value="0 0 0" />
+  <xacro:property name="link_hand_com_rpy" value="0 0 0" />
+  <xacro:property name="link_hand_mass" value="0.1" />
+  <xacro:property name="link_hand_Ixx" value="0.1" />
+  <xacro:property name="link_hand_Ixy" value="0.0" />
+  <xacro:property name="link_hand_Ixz" value="0.0" />
+  <xacro:property name="link_hand_Iyy" value="0.1" />
+  <xacro:property name="link_hand_Iyz" value="0.0" />
+  <xacro:property name="link_hand_Izz" value="0.1" />
+	<xacro:macro name="jaco_link" params="link_name link_mass Ixx Ixy Ixz Iyy Iyz Izz link_com_origin link_com_rpy">
 		<link name="${link_name}">
             <inertial>
-                <mass value="1"/>
-                <inertia ixx="0.1" ixy="0" ixz="0" iyy="0.1" iyz="0" izz="0.1"/>
-                <origin xyz="0.01 0.01 0.01" rpy="0 0 0"/>
+                <mass value="${link_mass}"/>
+                <inertia ixx="${Ixx}" ixy="${Ixy}" ixz="${Ixz}" iyy="${Iyy}" iyz="${Iyz}" izz="${Izz}"/>
+                <origin xyz="${link_com_origin}" rpy="${link_com_rpy}" />
             </inertial>
 			<visual>
@@ -130,10 +193,10 @@
 		</link>
 	</xacro:macro>
-	<xacro:macro name="jaco_link_4_5" params="link_name suffix">
+	<xacro:macro name="jaco_link_4_5" params="link_name suffix link_mass Ixx Ixy Ixz Iyy Iyz Izz link_com_origin link_com_rpy">
 		<link name="${link_name}_${suffix}">
             <inertial>
-                <mass value="0.5"/>
-                <inertia ixx="0.01" ixy="0" ixz="0" iyy="0.01" iyz="0" izz="0.01"/>
-                <origin/>
+                <mass value="${link_mass}"/>
+                <inertia ixx="${Ixx}" ixy="${Ixy}" ixz="${Ixz}" iyy="${Iyy}" iyz="${Iyz}" izz="${Izz}"/>
+                <origin xyz="${link_com_origin}" rpy="${link_com_rpy}" />
             </inertial>
 			<visual>
@@ -210,23 +273,23 @@
             </plugin>
         </gazebo>
-		<xacro:jaco_link link_name="${link_base}" />
+		<xacro:jaco_link link_name="${link_base}" link_mass="${link_base_mass}" Ixx="${link_base_Ixx}" Ixy="${link_base_Ixy}" Ixz="${link_base_Ixz}" Iyy="${link_base_Iyy}" Iyz="${link_base_Iyz}" Izz="${link_base_Izz}" link_com_origin="${link_base_com_xyz}" link_com_rpy="${link_base_com_rpy}" />
 		<xacro:jaco_joint joint_name="${joint_base}" type="fixed" parent="${parent}" child="${link_base}" joint_axis_xyz="${joint_base_axis_xyz}" joint_origin_xyz="${xyz}" joint_origin_rpy="${rpy}" lower_limit="-${J_LIM}" upper_limit="${J_LIM}" />
-		<xacro:jaco_link link_name="${link_1}" />
-		<xacro:jaco_joint joint_name="${joint_1}" type="revolute" parent="${link_base}" child="${link_1}" joint_axis_xyz="${joint_1_axis_xyz}" joint_origin_xyz="${joint_1_origin_xyz}" joint_origin_rpy="${joint_1_origin_rpy}" lower_limit="-${J_LIM}" upper_limit="${J_LIM}" />
+		<xacro:jaco_link link_name="${link_1}" link_mass="${link_1_mass}" Ixx="${link_1_Ixx}" Ixy="${link_1_Ixy}" Ixz="${link_1_Ixz}" Iyy="${link_1_Iyy}" Iyz="${link_1_Iyz}" Izz="${link_1_Izz}" link_com_origin="${link_1_com_xyz}" link_com_rpy="${link_1_com_rpy}" />
+		<xacro:jaco_joint joint_name="${joint_1}" type="revolute" parent="${link_base}" child="${link_1}" joint_axis_xyz="${joint_1_axis_xyz}" joint_origin_xyz="${joint_1_origin_xyz}" joint_origin_rpy="${joint_1_origin_rpy}" lower_limit="-${J_LIM}" upper_limit="${J_LIM}"/>
         <xacro:jaco_transmission joint_name="${joint_1}" />
-		<xacro:jaco_link link_name="${link_2}" />
-		<xacro:jaco_joint joint_name="${joint_2}" type="revolute" parent="${link_1}" child="${link_2}" joint_axis_xyz="${joint_2_axis_xyz}" joint_origin_xyz="${joint_2_origin_xyz}" joint_origin_rpy="${joint_2_origin_rpy}" lower_limit="0" upper_limit="${J_LIM}" />
+		<xacro:jaco_link link_name="${link_2}" link_mass="${link_2_mass}" Ixx="${link_2_Ixx}" Ixy="${link_2_Ixy}" Ixz="${link_2_Ixz}" Iyy="${link_2_Iyy}" Iyz="${link_2_Iyz}" Izz="${link_2_Izz}" link_com_origin="${link_2_com_xyz}" link_com_rpy="${link_2_com_rpy}" />
+		<xacro:jaco_joint joint_name="${joint_2}" type="revolute" parent="${link_1}" child="${link_2}" joint_axis_xyz="${joint_2_axis_xyz}" joint_origin_xyz="${joint_2_origin_xyz}" joint_origin_rpy="${joint_2_origin_rpy}" lower_limit="0" upper_limit="${J_LIM}"  />
         <xacro:jaco_transmission joint_name="${joint_2}" />
-		<xacro:jaco_link link_name="${link_3}" />
-		<xacro:jaco_joint joint_name="${joint_3}" type="revolute" parent="${link_2}" child="${link_3}" joint_axis_xyz="${joint_3_axis_xyz}" joint_origin_xyz="${joint_3_origin_xyz}" joint_origin_rpy="${joint_3_origin_rpy}" lower_limit="0" upper_limit="${J_LIM}" />
+		<xacro:jaco_link link_name="${link_3}" link_mass="${link_3_mass}" Ixx="${link_3_Ixx}" Ixy="${link_3_Ixy}" Ixz="${link_3_Ixz}" Iyy="${link_3_Iyy}" Iyz="${link_3_Iyz}" Izz="${link_3_Izz}" link_com_origin="${link_3_com_xyz}" link_com_rpy="${link_3_com_rpy}" />
+		<xacro:jaco_joint joint_name="${joint_3}" type="revolute" parent="${link_2}" child="${link_3}" joint_axis_xyz="${joint_3_axis_xyz}" joint_origin_xyz="${joint_3_origin_xyz}" joint_origin_rpy="${joint_3_origin_rpy}" lower_limit="0" upper_limit="${J_LIM}"  />
         <xacro:jaco_transmission joint_name="${joint_3}" />
-		<xacro:jaco_link_4_5 link_name="${link}" suffix="4"/>
-		<xacro:jaco_joint joint_name="${joint_4}" type="revolute" parent="${link_3}" child="${link}_4" joint_axis_xyz="${joint_4_axis_xyz}" joint_origin_xyz="${joint_4_origin_xyz}" joint_origin_rpy="${joint_4_origin_rpy}" lower_limit="-${J_LIM}" upper_limit="${J_LIM}" />
+		<xacro:jaco_link_4_5 link_name="${link}" suffix="4" link_mass="${link_4_mass}" Ixx="${link_4_Ixx}" Ixy="${link_4_Ixy}" Ixz="${link_4_Ixz}" Iyy="${link_4_Iyy}" Iyz="${link_4_Iyz}" Izz="${link_4_Izz}" link_com_origin="${link_4_com_xyz}" link_com_rpy="${link_4_com_rpy}"/>
+		<xacro:jaco_joint joint_name="${joint_4}" type="revolute" parent="${link_3}" child="${link}_4" joint_axis_xyz="${joint_4_axis_xyz}" joint_origin_xyz="${joint_4_origin_xyz}" joint_origin_rpy="${joint_4_origin_rpy}" lower_limit="-${J_LIM}" upper_limit="${J_LIM}"  />
         <xacro:jaco_transmission joint_name="${joint_4}" />
-		<xacro:jaco_link_4_5 link_name="${link}" suffix="5"/>
-		<xacro:jaco_joint joint_name="${joint_5}" type="revolute" parent="${link}_4" child="${link}_5" joint_axis_xyz="${joint_5_axis_xyz}" joint_origin_xyz="${joint_5_origin_xyz}" joint_origin_rpy="${joint_5_origin_rpy}" lower_limit="-${J_LIM}" upper_limit="${J_LIM}" />
+		<xacro:jaco_link_4_5 link_name="${link}" suffix="5" link_mass="${link_5_mass}" Ixx="${link_5_Ixx}" Ixy="${link_5_Ixy}" Ixz="${link_5_Ixz}" Iyy="${link_5_Iyy}" Iyz="${link_5_Iyz}" Izz="${link_5_Izz}" link_com_origin="${link_5_com_xyz}" link_com_rpy="${link_5_com_rpy}"/>
+		<xacro:jaco_joint joint_name="${joint_5}" type="revolute" parent="${link}_4" child="${link}_5" joint_axis_xyz="${joint_5_axis_xyz}" joint_origin_xyz="${joint_5_origin_xyz}" joint_origin_rpy="${joint_5_origin_rpy}" lower_limit="-${J_LIM}" upper_limit="${J_LIM}"/>
         <xacro:jaco_transmission joint_name="${joint_5}" />
-		<xacro:jaco_link link_name="${link_hand}" />
-		<xacro:jaco_joint joint_name="${joint_6}" type="revolute" parent="${link}_5" child="${link_hand}" joint_axis_xyz="${joint_6_axis_xyz}" joint_origin_xyz="${joint_6_origin_xyz}" joint_origin_rpy="${joint_6_origin_rpy}" lower_limit="-${J_LIM}" upper_limit="${J_LIM}" />
+		<xacro:jaco_link link_name="${link_hand}" link_mass="${link_hand_mass}" Ixx="${link_hand_Ixx}" Ixy="${link_hand_Ixy}" Ixz="${link_hand_Ixz}" Iyy="${link_hand_Iyy}" Iyz="${link_hand_Iyz}" Izz="${link_hand_Izz}" link_com_origin="${link_hand_com_xyz}" link_com_rpy="${link_hand_com_rpy}"/>
+		<xacro:jaco_joint joint_name="${joint_6}" type="revolute" parent="${link}_5" child="${link_hand}" joint_axis_xyz="${joint_6_axis_xyz}" joint_origin_xyz="${joint_6_origin_xyz}" joint_origin_rpy="${joint_6_origin_rpy}" lower_limit="-${J_LIM}" upper_limit="${J_LIM}"/>
         <xacro:jaco_transmission joint_name="${joint_6}" />
 		<xacro:jaco_ring_cover suffix="1" size="large"/>

Commit message: some minor additions still wrong inertias

File: jaco_description/urdf/jaco_arm.urdf.xacro (robot description, xacro)
@@ -88,65 +88,65 @@
   <xacro:property name="link_base_com_xyz" value="0 0 0" />
   <xacro:property name="link_base_com_rpy" value="0 0 0" />
-  <xacro:property name="link_base_mass" value="0.1" />
+  <xacro:property name="link_base_mass" value="0.0" />
   <xacro:property name="link_base_Ixx" value="0.1" />
-  <xacro:property name="link_base_Ixy" value="0.0" />
-  <xacro:property name="link_base_Ixz" value="0.0" />
-  <xacro:property name="link_base_Iyy" value="0.1" />
-  <xacro:property name="link_base_Iyz" value="0.0" />
-  <xacro:property name="link_base_Izz" value="0.1" />
-  <xacro:property name="link_1_com_xyz" value="0 0 0" />
+  <xacro:property name="link_base_Ixy" value="0.2" />
+  <xacro:property name="link_base_Ixz" value="0.3" />
+  <xacro:property name="link_base_Iyy" value="0.4" />
+  <xacro:property name="link_base_Iyz" value="0.5" />
+  <xacro:property name="link_base_Izz" value="0.6" />
+  <xacro:property name="link_1_com_xyz" value="0 0.0086 -0.1064" />
   <xacro:property name="link_1_com_rpy" value="0 0 0" />
-  <xacro:property name="link_1_mass" value="0.1" />
-  <xacro:property name="link_1_Ixx" value="0.1" />
-  <xacro:property name="link_1_Ixy" value="0.0" />
-  <xacro:property name="link_1_Ixz" value="0.0" />
-  <xacro:property name="link_1_Iyy" value="0.1" />
-  <xacro:property name="link_1_Iyz" value="0.0" />
-  <xacro:property name="link_1_Izz" value="0.1" />
-  <xacro:property name="link_2_com_xyz" value="0 0 0" />
+  <xacro:property name="link_1_mass" value="0.7417" />
+  <xacro:property name="link_1_Ixx" value="0.0002" />
+  <xacro:property name="link_1_Ixy" value="-0.0003" />
+  <xacro:property name="link_1_Ixz" value="-0.0003" />
+  <xacro:property name="link_1_Iyy" value="0.0431" />
+  <xacro:property name="link_1_Iyz" value="0.0003" />
+  <xacro:property name="link_1_Izz" value="0.0004" />
+  <xacro:property name="link_2_com_xyz" value="0.2452 0 -0.0921" />
   <xacro:property name="link_2_com_rpy" value="0 0 0" />
-  <xacro:property name="link_2_mass" value="0.1" />
-  <xacro:property name="link_2_Ixx" value="0.1" />
-  <xacro:property name="link_2_Ixy" value="0.0" />
-  <xacro:property name="link_2_Ixz" value="0.0" />
-  <xacro:property name="link_2_Iyy" value="0.1" />
-  <xacro:property name="link_2_Iyz" value="0.0" />
-  <xacro:property name="link_2_Izz" value="0.1" />
-  <xacro:property name="link_3_com_xyz" value="0 0 0" />
+  <xacro:property name="link_2_mass" value="0.9977" />
+  <xacro:property name="link_2_Ixx" value="-0.0091" />
+  <xacro:property name="link_2_Ixy" value="-0.0461" />
+  <xacro:property name="link_2_Ixz" value="-0.0275" />
+  <xacro:property name="link_2_Iyy" value="-0.0421" />
+  <xacro:property name="link_2_Iyz" value="-0.0461" />
+  <xacro:property name="link_2_Izz" value="-0.0326" />
+  <xacro:property name="link_3_com_xyz" value="0.1624 0.0 -0.0135" />
   <xacro:property name="link_3_com_rpy" value="0 0 0" />
-  <xacro:property name="link_3_mass" value="0.1" />
-  <xacro:property name="link_3_Ixx" value="0.1" />
-  <xacro:property name="link_3_Ixy" value="0.0" />
-  <xacro:property name="link_3_Ixz" value="0.0" />
-  <xacro:property name="link_3_Iyy" value="0.1" />
-  <xacro:property name="link_3_Iyz" value="0.0" />
-  <xacro:property name="link_3_Izz" value="0.1" />
-  <xacro:property name="link_4_com_xyz" value="0 0 0" />
+  <xacro:property name="link_3_mass" value="0.7847" />
+  <xacro:property name="link_3_Ixx" value=" 0.0003" />
+  <xacro:property name="link_3_Ixy" value="-0.0028" />
+  <xacro:property name="link_3_Ixz" value="-0.0026" />
+  <xacro:property name="link_3_Iyy" value="-0.0021" />
+  <xacro:property name="link_3_Iyz" value="-0.0028" />
+  <xacro:property name="link_3_Izz" value="-0.0020" />
+  <xacro:property name="link_4_com_xyz" value="0.0253 0.0000 -0.0585" />
   <xacro:property name="link_4_com_rpy" value="0 0 0" />
-  <xacro:property name="link_4_mass" value="0.1" />
-  <xacro:property name="link_4_Ixx" value="0.1" />
-  <xacro:property name="link_4_Ixy" value="0.0" />
-  <xacro:property name="link_4_Ixz" value="0.0" />
-  <xacro:property name="link_4_Iyy" value="0.1" />
-  <xacro:property name="link_4_Iyz" value="0.0" />
-  <xacro:property name="link_4_Izz" value="0.1" />
-  <xacro:property name="link_5_com_xyz" value="0 0 0" />
+  <xacro:property name="link_4_mass" value="0.6426" />
+  <xacro:property name="link_4_Ixx" value=" 0.0002" />
+  <xacro:property name="link_4_Ixy" value="-0.0001" />
+  <xacro:property name="link_4_Ixz" value="-0.0001" />
+  <xacro:property name="link_4_Iyy" value=" 0.0002" />
+  <xacro:property name="link_4_Iyz" value="-0.0001" />
+  <xacro:property name="link_4_Izz" value=" 0.0003" />
+  <xacro:property name="link_5_com_xyz" value="0.0253 0.0000 -0.0585" />
   <xacro:property name="link_5_com_rpy" value="0 0 0" />
-  <xacro:property name="link_5_mass" value="0.1" />
-  <xacro:property name="link_5_Ixx" value="0.1" />
-  <xacro:property name="link_5_Ixy" value="0.0" />
-  <xacro:property name="link_5_Ixz" value="0.0" />
-  <xacro:property name="link_5_Iyy" value="0.1" />
-  <xacro:property name="link_5_Iyz" value="0.0" />
-  <xacro:property name="link_5_Izz" value="0.1" />
-  <xacro:property name="link_hand_com_xyz" value="0 0 0" />
+  <xacro:property name="link_5_mass" value="0.6426" />
+  <xacro:property name="link_5_Ixx" value=" 0.0002" />
+  <xacro:property name="link_5_Ixy" value="-0.0001" />
+  <xacro:property name="link_5_Ixz" value="-0.0001" />
+  <xacro:property name="link_5_Iyy" value=" 0.0002" />
+  <xacro:property name="link_5_Iyz" value="-0.0001" />
+  <xacro:property name="link_5_Izz" value=" 0.0003" />
+  <xacro:property name="link_hand_com_xyz" value="0.0068 0 -0.0822" />
   <xacro:property name="link_hand_com_rpy" value="0 0 0" />
-  <xacro:property name="link_hand_mass" value="0.1" />
-  <xacro:property name="link_hand_Ixx" value="0.1" />
-  <xacro:property name="link_hand_Ixy" value="0.0" />
-  <xacro:property name="link_hand_Ixz" value="0.0" />
-  <xacro:property name="link_hand_Iyy" value="0.1" />
-  <xacro:property name="link_hand_Iyz" value="0.0" />
-  <xacro:property name="link_hand_Izz" value="0.1" />
+  <xacro:property name="link_hand_mass" value="0.7270" />
+  <xacro:property name="link_hand_Ixx" value="-0.0049 " />
+  <xacro:property name="link_hand_Ixy" value="-0.0049" />
+  <xacro:property name="link_hand_Ixz" value="-0.0054" />
+  <xacro:property name="link_hand_Iyy" value="-0.0049" />
+  <xacro:property name="link_hand_Iyz" value="-0.0050" />
+  <xacro:property name="link_hand_Izz" value="-0.000008" />
 	<xacro:macro name="jaco_link" params="link_name link_mass Ixx Ixy Ixz Iyy Iyz Izz link_com_origin link_com_rpy">
 		<link name="${link_name}">
