Commit message: renamed jaco_description to jaco2_description

File: jaco2_description/robots/cylinder_arm.urdf.xacro (robot description, xacro)
@@ -13,5 +13,5 @@
 	xmlns:physics="http://playerstage.sourceforge.net/gazebo/xmlschema/#physics"
 	xmlns:xacro="http://ros.org/wiki/xacro" name="jaco">
-	<xacro:include filename="$(find jaco_description)/urdf/jaco_arm.urdf.xacro" />
+	<xacro:include filename="$(find jaco2_description)/urdf/jaco_arm.urdf.xacro" />
 	<link name="root">
 		<visual>

File: jaco2_description/robots/standalone_arm.urdf.xacro (robot description, xacro)
@@ -13,5 +13,5 @@
 	xmlns:physics="http://playerstage.sourceforge.net/gazebo/xmlschema/#physics"
 	xmlns:xacro="http://ros.org/wiki/xacro" name="jaco">
-	<xacro:include filename="$(find jaco_description)/urdf/jaco_arm.urdf.xacro" />
+	<xacro:include filename="$(find jaco2_description)/urdf/jaco_arm.urdf.xacro" />
 	<link name="root">
 		<visual>

File: jaco2_description/urdf/jaco_arm.urdf.xacro (robot description, xacro)
@@ -158,5 +158,5 @@
 			<visual>
 				<geometry>
-					<mesh scale="${M_SCALE} ${M_SCALE} ${M_SCALE}" filename="package://jaco_description/meshes/${link_name}.min.dae" />
+					<mesh scale="${M_SCALE} ${M_SCALE} ${M_SCALE}" filename="package://jaco2_description/meshes/${link_name}.min.dae" />
 				</geometry>
 				<material name="carbon_fiber">
@@ -166,5 +166,5 @@
 			<collision>
 				<geometry>
-					<mesh scale="${M_SCALE} ${M_SCALE} ${M_SCALE}" filename="package://jaco_description/meshes/${link_name}.stl" />
+					<mesh scale="${M_SCALE} ${M_SCALE} ${M_SCALE}" filename="package://jaco2_description/meshes/${link_name}.stl" />
 				</geometry>
 			</collision>
@@ -180,5 +180,5 @@
 			<visual>
 				<geometry>
-					<mesh scale="${M_SCALE} ${M_SCALE} ${M_SCALE}" filename="package://jaco_description/meshes/${link_name}.min.dae" />
+					<mesh scale="${M_SCALE} ${M_SCALE} ${M_SCALE}" filename="package://jaco2_description/meshes/${link_name}.min.dae" />
 				</geometry>
 				<material name="carbon_fiber">
@@ -188,5 +188,5 @@
 			<collision>
 				<geometry>
-					<mesh scale="${M_SCALE} ${M_SCALE} ${M_SCALE}" filename="package://jaco_description/meshes/${link_name}.stl" />
+					<mesh scale="${M_SCALE} ${M_SCALE} ${M_SCALE}" filename="package://jaco2_description/meshes/${link_name}.stl" />
 				</geometry>
 			</collision>
@@ -202,5 +202,5 @@
 			<visual>
 				<geometry>
-					<mesh scale="${M_SCALE} ${M_SCALE} ${M_SCALE}" filename="package://jaco_description/meshes/${link_name}_4_5.min.dae" />
+					<mesh scale="${M_SCALE} ${M_SCALE} ${M_SCALE}" filename="package://jaco2_description/meshes/${link_name}_4_5.min.dae" />
 				</geometry>
 				<material name="carbon_fiber">
@@ -210,5 +210,5 @@
 			<collision>
 				<geometry>
-					<mesh scale="${M_SCALE} ${M_SCALE} ${M_SCALE}" filename="package://jaco_description/meshes/${link_name}_4_5.stl" />
+					<mesh scale="${M_SCALE} ${M_SCALE} ${M_SCALE}" filename="package://jaco2_description/meshes/${link_name}_4_5.stl" />
 				</geometry>
 			</collision>
@@ -224,5 +224,5 @@
 			<visual>
 				<geometry>
-					<mesh scale="${M_SCALE} ${M_SCALE} ${M_SCALE}" filename="package://jaco_description/meshes/jaco_${size}_ring_cover.min.dae" />
+					<mesh scale="${M_SCALE} ${M_SCALE} ${M_SCALE}" filename="package://jaco2_description/meshes/jaco_${size}_ring_cover.min.dae" />
 				</geometry>
 				<material name="carbon_fiber">
@@ -232,5 +232,5 @@
 			<collision>
 				<geometry>
-					<mesh scale="${M_SCALE} ${M_SCALE} ${M_SCALE}" filename="package://jaco_description/meshes/jaco_${size}_ring_cover.stl" />
+					<mesh scale="${M_SCALE} ${M_SCALE} ${M_SCALE}" filename="package://jaco2_description/meshes/jaco_${size}_ring_cover.stl" />
 				</geometry>
 			</collision>
