Commit message: Adjust gain p2p controller and modify config files

File: jaco2_description/urdf/jaco_arm_with_realsense.urdf.xacro (robot description, xacro)
@@ -30,6 +30,6 @@
   <xacro:property name="joint_1_origin_xyz" value="0 0 0.15675" />
   <xacro:property name="joint_1_origin_rpy" value="${M_PI} 0 0" />
-  <xacro:property name="joint_1_lower_limit" value="${-2*M_PI}" />
-  <xacro:property name="joint_1_upper_limit" value="${2*M_PI}" />
+  <xacro:property name="joint_1_lower_limit" value="${-M_PI}" />
+  <xacro:property name="joint_1_upper_limit" value="${M_PI}" />
   <xacro:property name="joint_2" value="jaco_joint_2" />
   <xacro:property name="joint_2_axis_xyz" value="0 0 1" />
@@ -48,18 +48,18 @@
   <xacro:property name="joint_4_origin_xyz" value="0.2073 0 -0.0114" />
   <xacro:property name="joint_4_origin_rpy" value="0 -${M_PI/2} 0" />
-  <xacro:property name="joint_4_lower_limit" value="${-2*M_PI}" />
-  <xacro:property name="joint_4_upper_limit" value="${2*M_PI}" />
+  <xacro:property name="joint_4_lower_limit" value="${-M_PI}" />
+  <xacro:property name="joint_4_upper_limit" value="${M_PI}" />
   <xacro:property name="joint_5" value="jaco_joint_5" />
   <xacro:property name="joint_5_axis_xyz" value="0 0 1" />
   <xacro:property name="joint_5_origin_xyz" value="0.03705 0 -0.0641725" />
   <xacro:property name="joint_5_origin_rpy" value="0 ${M_PI/180*60} ${M_PI}" /> <!-- maybe 55 degrees, Advanded user guide specifys 60 ...-->
-  <xacro:property name="joint_5_lower_limit" value="${-2*M_PI}" />
-  <xacro:property name="joint_5_upper_limit" value="${2*M_PI}" />
+  <xacro:property name="joint_5_lower_limit" value="${-M_PI}" />
+  <xacro:property name="joint_5_upper_limit" value="${M_PI}" />
   <xacro:property name="joint_6" value="jaco_joint_6" />
   <xacro:property name="joint_6_axis_xyz" value="0 0 1" />
   <xacro:property name="joint_6_origin_xyz" value="0.03705 0 -0.0641725" />
   <xacro:property name="joint_6_origin_rpy" value="0 ${M_PI/180*60} ${M_PI}" /> <!-- maybe 55 degrees, Advanded user guide specifys 60 ...-->
-  <xacro:property name="joint_6_lower_limit" value="${-2*M_PI}" />
-  <xacro:property name="joint_6_upper_limit" value="${2*M_PI}" />
+  <xacro:property name="joint_6_lower_limit" value="${-M_PI}" />
+  <xacro:property name="joint_6_upper_limit" value="${M_PI}" />
   <xacro:property name="joint_finger_1" value="jaco_joint_finger_1" />
   <xacro:property name="joint_finger_1_axis_xyz" value="0 0 1" />

Commit message: Enhance trajectory gains for jaco 22

File: jaco2_description/urdf/jaco_arm_with_realsense.urdf.xacro (robot description, xacro)
@@ -152,13 +152,13 @@
   <xacro:property name="link_5_Iyz" value=" 0.0000" />
   <xacro:property name="link_5_Izz" value=" 0.0003" />
-  <xacro:property name="link_hand_com_xyz" value="0.0068 0 -0.0822" />
+  <xacro:property name="link_hand_com_xyz" value="0.0058 0.0104 -0.0703" />
   <xacro:property name="link_hand_com_rpy" value="0 0 0" />
-  <xacro:property name="link_hand_mass" value="0.7270" />
-  <xacro:property name="link_hand_Ixx" value=" 0.0050" />
-  <xacro:property name="link_hand_Ixy" value=" 0.0000" />
-  <xacro:property name="link_hand_Ixz" value=" 0.0004" />
-  <xacro:property name="link_hand_Iyy" value=" 0.0050" />
-  <xacro:property name="link_hand_Iyz" value=" 0.0000" />
-  <xacro:property name="link_hand_Izz" value=" 0.0001" />
+  <xacro:property name="link_hand_mass" value="0.8579" />
+  <xacro:property name="link_hand_Ixx" value=" 0.0091" />
+  <xacro:property name="link_hand_Ixy" value=" 0.0001" />
+  <xacro:property name="link_hand_Ixz" value=" 0.0041" />
+  <xacro:property name="link_hand_Iyy" value=" 0.0185" />
+  <xacro:property name="link_hand_Iyz" value=" 0.0001" />
+  <xacro:property name="link_hand_Izz" value=" 0.0126" />
 	<xacro:macro name="jaco_link" params="link_name link_mass Ixx Ixy Ixz Iyy Iyz Izz link_com_origin link_com_rpy">
 		<link name="${link_name}">

Commit message: Add config for inertia parameters jaco2

File: jaco2_description/urdf/jaco_arm_with_realsense.urdf.xacro (robot description, xacro)
@@ -152,13 +152,13 @@
   <xacro:property name="link_5_Iyz" value=" 0.0000" />
   <xacro:property name="link_5_Izz" value=" 0.0003" />
-  <xacro:property name="link_hand_com_xyz" value="0.0058 0.0104 -0.0703" />
+  <xacro:property name="link_hand_com_xyz" value="0.0058 0.0091 -0.0688" />
   <xacro:property name="link_hand_com_rpy" value="0 0 0" />
   <xacro:property name="link_hand_mass" value="0.8579" />
-  <xacro:property name="link_hand_Ixx" value=" 0.0091" />
-  <xacro:property name="link_hand_Ixy" value=" 0.0001" />
-  <xacro:property name="link_hand_Ixz" value=" 0.0041" />
-  <xacro:property name="link_hand_Iyy" value=" 0.0185" />
+  <xacro:property name="link_hand_Ixx" value=" 0.0093" />
+  <xacro:property name="link_hand_Ixy" value=" 0.0000" />
+  <xacro:property name="link_hand_Ixz" value=" 0.0042" />
+  <xacro:property name="link_hand_Iyy" value=" 0.0182" />
   <xacro:property name="link_hand_Iyz" value=" 0.0001" />
-  <xacro:property name="link_hand_Izz" value=" 0.0126" />
+  <xacro:property name="link_hand_Izz" value=" 0.0130" />
 	<xacro:macro name="jaco_link" params="link_name link_mass Ixx Ixy Ixz Iyy Iyz Izz link_com_origin link_com_rpy">
 		<link name="${link_name}">

Commit message: Reduce longest_valid_segment_fraction seems to be saver; Improve config for jaco2_realsense

File: jaco2_description/urdf/jaco_arm_with_realsense.urdf.xacro (robot description, xacro)
@@ -30,6 +30,6 @@
   <xacro:property name="joint_1_origin_xyz" value="0 0 0.15675" />
   <xacro:property name="joint_1_origin_rpy" value="${M_PI} 0 0" />
-  <xacro:property name="joint_1_lower_limit" value="${-M_PI}" />
-  <xacro:property name="joint_1_upper_limit" value="${M_PI}" />
+  <xacro:property name="joint_1_lower_limit" value="${0.5*M_PI}" />
+  <xacro:property name="joint_1_upper_limit" value="${2.5*M_PI}" />
   <xacro:property name="joint_2" value="jaco_joint_2" />
   <xacro:property name="joint_2_axis_xyz" value="0 0 1" />
@@ -48,6 +48,6 @@
   <xacro:property name="joint_4_origin_xyz" value="0.2073 0 -0.0114" />
   <xacro:property name="joint_4_origin_rpy" value="0 -${M_PI/2} 0" />
-  <xacro:property name="joint_4_lower_limit" value="${-M_PI}" />
-  <xacro:property name="joint_4_upper_limit" value="${M_PI}" />
+  <xacro:property name="joint_4_lower_limit" value="${0.5*M_PI}" />
+  <xacro:property name="joint_4_upper_limit" value="${2.5*M_PI}" />
   <xacro:property name="joint_5" value="jaco_joint_5" />
   <xacro:property name="joint_5_axis_xyz" value="0 0 1" />

Commit message: Send geometry_msgs/Twist to to topic

File: jaco2_description/urdf/jaco_arm_with_realsense.urdf.xacro (robot description, xacro)
@@ -200,5 +200,5 @@
 			<collision>
 				<geometry>
-					<mesh scale="${M_SCALE} ${M_SCALE} ${M_SCALE}" filename="package://jaco2_description/meshes/${file}_convex_hull.stl" />
+					<mesh scale="${M_SCALE} ${M_SCALE} ${M_SCALE}" filename="package://jaco2_description/meshes/${file}.stl" />
 				</geometry>
 			</collision>
@@ -324,5 +324,5 @@
 		<xacro:jaco_joint joint_name="${joint_5}" type="revolute" parent="${link}_4" child="${link}_5" joint_axis_xyz="${joint_5_axis_xyz}" joint_origin_xyz="${joint_5_origin_xyz}" joint_origin_rpy="${joint_5_origin_rpy}" lower_limit="${joint_5_lower_limit}" upper_limit="${joint_5_upper_limit}"/>
         <xacro:jaco_transmission joint_name="${joint_5}" />
-		<xacro:jaco_eeff_link link_name="${link_hand}" file="jaco_hand_with_realsense" link_mass="${link_hand_mass}" Ixx="${link_hand_Ixx}" Ixy="${link_hand_Ixy}" Ixz="${link_hand_Ixz}" Iyy="${link_hand_Iyy}" Iyz="${link_hand_Iyz}" Izz="${link_hand_Izz}" link_com_origin="${link_hand_com_xyz}" link_com_rpy="${link_hand_com_rpy}"/>
+		<xacro:jaco_eeff_link link_name="${link_hand}" file="sick_hand_notloesung_inch" link_mass="${link_hand_mass}" Ixx="${link_hand_Ixx}" Ixy="${link_hand_Ixy}" Ixz="${link_hand_Ixz}" Iyy="${link_hand_Iyy}" Iyz="${link_hand_Iyz}" Izz="${link_hand_Izz}" link_com_origin="${link_hand_com_xyz}" link_com_rpy="${link_hand_com_rpy}"/>
 		<xacro:jaco_joint joint_name="${joint_6}" type="revolute" parent="${link}_5" child="${link_hand}" joint_axis_xyz="${joint_6_axis_xyz}" joint_origin_xyz="${joint_6_origin_xyz}" joint_origin_rpy="${joint_6_origin_rpy}" lower_limit="${joint_6_lower_limit}" upper_limit="${joint_6_upper_limit}"/>
         <xacro:jaco_transmission joint_name="${joint_6}" />
