Commit message: Add a view changes

File: jaco2_description/urdf/jaco_arm.urdf.xacro (robot description, xacro)
@@ -30,24 +30,36 @@
   <xacro:property name="joint_1_origin_xyz" value="0 0 0.15675" />
   <xacro:property name="joint_1_origin_rpy" value="${M_PI} 0 0" />
+  <xacro:property name="joint_1_lower_limit" value="${-2*M_PI}" />
+  <xacro:property name="joint_1_upper_limit" value="${2*M_PI}" />
   <xacro:property name="joint_2" value="jaco_joint_2" />
   <xacro:property name="joint_2_axis_xyz" value="0 0 1" />
   <xacro:property name="joint_2_origin_xyz" value="0 0.0016 -0.11875" />
   <xacro:property name="joint_2_origin_rpy" value="-${M_PI/2} -${M_PI/2} 0" />
+  <xacro:property name="joint_2_lower_limit" value="${M_PI/180*50}" />
+  <xacro:property name="joint_2_upper_limit" value="${M_PI/180*310}" />
   <xacro:property name="joint_3" value="jaco_joint_3" />
   <xacro:property name="joint_3_axis_xyz" value="0 0 1" />
   <xacro:property name="joint_3_origin_xyz" value="0.41 0 0" />
   <xacro:property name="joint_3_origin_rpy" value="${M_PI} 0 ${M_PI}" />
+  <xacro:property name="joint_3_lower_limit" value="${M_PI/180*19}" />
+  <xacro:property name="joint_3_upper_limit" value="${M_PI/180*341}" />
   <xacro:property name="joint_4" value="jaco_joint_4" />
   <xacro:property name="joint_4_axis_xyz" value="0 0 1" />
   <xacro:property name="joint_4_origin_xyz" value="0.2073 0 -0.0114" />
   <xacro:property name="joint_4_origin_rpy" value="0 -${M_PI/2} 0" />
+  <xacro:property name="joint_4_lower_limit" value="${-2*M_PI}" />
+  <xacro:property name="joint_4_upper_limit" value="${2*M_PI}" />
   <xacro:property name="joint_5" value="jaco_joint_5" />
   <xacro:property name="joint_5_axis_xyz" value="0 0 1" />
   <xacro:property name="joint_5_origin_xyz" value="0.03705 0 -0.0641725" />
   <xacro:property name="joint_5_origin_rpy" value="0 ${M_PI/180*60} ${M_PI}" /> <!-- maybe 55 degrees, Advanded user guide specifys 60 ...-->
+  <xacro:property name="joint_5_lower_limit" value="${-2*M_PI}" />
+  <xacro:property name="joint_5_upper_limit" value="${2*M_PI}" />
   <xacro:property name="joint_6" value="jaco_joint_6" />
   <xacro:property name="joint_6_axis_xyz" value="0 0 1" />
   <xacro:property name="joint_6_origin_xyz" value="0.03705 0 -0.0641725" />
   <xacro:property name="joint_6_origin_rpy" value="0 ${M_PI/180*60} ${M_PI}" /> <!-- maybe 55 degrees, Advanded user guide specifys 60 ...-->
+  <xacro:property name="joint_6_lower_limit" value="${-2*M_PI}" />
+  <xacro:property name="joint_6_upper_limit" value="${2*M_PI}" />
   <xacro:property name="joint_finger_1" value="jaco_joint_finger_1" />
   <xacro:property name="joint_finger_1_axis_xyz" value="0 0 1" />
@@ -276,20 +288,20 @@
 		<xacro:jaco_joint joint_name="${joint_base}" type="fixed" parent="${parent}" child="${link_base}" joint_axis_xyz="${joint_base_axis_xyz}" joint_origin_xyz="${xyz}" joint_origin_rpy="${rpy}" lower_limit="-${J_LIM}" upper_limit="${J_LIM}" />
 		<xacro:jaco_link link_name="${link_1}" link_mass="${link_1_mass}" Ixx="${link_1_Ixx}" Ixy="${link_1_Ixy}" Ixz="${link_1_Ixz}" Iyy="${link_1_Iyy}" Iyz="${link_1_Iyz}" Izz="${link_1_Izz}" link_com_origin="${link_1_com_xyz}" link_com_rpy="${link_1_com_rpy}" />
-		<xacro:jaco_joint joint_name="${joint_1}" type="revolute" parent="${link_base}" child="${link_1}" joint_axis_xyz="${joint_1_axis_xyz}" joint_origin_xyz="${joint_1_origin_xyz}" joint_origin_rpy="${joint_1_origin_rpy}" lower_limit="-${J_LIM}" upper_limit="${J_LIM}"/>
+		<xacro:jaco_joint joint_name="${joint_1}" type="revolute" parent="${link_base}" child="${link_1}" joint_axis_xyz="${joint_1_axis_xyz}" joint_origin_xyz="${joint_1_origin_xyz}" joint_origin_rpy="${joint_1_origin_rpy}" lower_limit="${joint_1_lower_limit}" upper_limit="${joint_1_upper_limit}"/>
         <xacro:jaco_transmission joint_name="${joint_1}" />
 		<xacro:jaco_link link_name="${link_2}" link_mass="${link_2_mass}" Ixx="${link_2_Ixx}" Ixy="${link_2_Ixy}" Ixz="${link_2_Ixz}" Iyy="${link_2_Iyy}" Iyz="${link_2_Iyz}" Izz="${link_2_Izz}" link_com_origin="${link_2_com_xyz}" link_com_rpy="${link_2_com_rpy}" />
-		<xacro:jaco_joint joint_name="${joint_2}" type="revolute" parent="${link_1}" child="${link_2}" joint_axis_xyz="${joint_2_axis_xyz}" joint_origin_xyz="${joint_2_origin_xyz}" joint_origin_rpy="${joint_2_origin_rpy}" lower_limit="0" upper_limit="${J_LIM}"  />
+		<xacro:jaco_joint joint_name="${joint_2}" type="revolute" parent="${link_1}" child="${link_2}" joint_axis_xyz="${joint_2_axis_xyz}" joint_origin_xyz="${joint_2_origin_xyz}" joint_origin_rpy="${joint_2_origin_rpy}" lower_limit="${joint_2_lower_limit}" upper_limit="${joint_2_upper_limit}"  />
         <xacro:jaco_transmission joint_name="${joint_2}" />
 		<xacro:jaco_link link_name="${link_3}" link_mass="${link_3_mass}" Ixx="${link_3_Ixx}" Ixy="${link_3_Ixy}" Ixz="${link_3_Ixz}" Iyy="${link_3_Iyy}" Iyz="${link_3_Iyz}" Izz="${link_3_Izz}" link_com_origin="${link_3_com_xyz}" link_com_rpy="${link_3_com_rpy}" />
-		<xacro:jaco_joint joint_name="${joint_3}" type="revolute" parent="${link_2}" child="${link_3}" joint_axis_xyz="${joint_3_axis_xyz}" joint_origin_xyz="${joint_3_origin_xyz}" joint_origin_rpy="${joint_3_origin_rpy}" lower_limit="0" upper_limit="${J_LIM}"  />
+		<xacro:jaco_joint joint_name="${joint_3}" type="revolute" parent="${link_2}" child="${link_3}" joint_axis_xyz="${joint_3_axis_xyz}" joint_origin_xyz="${joint_3_origin_xyz}" joint_origin_rpy="${joint_3_origin_rpy}" lower_limit="${joint_3_lower_limit}" upper_limit="${joint_3_upper_limit}"  />
         <xacro:jaco_transmission joint_name="${joint_3}" />
 		<xacro:jaco_link_4_5 link_name="${link}" suffix="4" link_mass="${link_4_mass}" Ixx="${link_4_Ixx}" Ixy="${link_4_Ixy}" Ixz="${link_4_Ixz}" Iyy="${link_4_Iyy}" Iyz="${link_4_Iyz}" Izz="${link_4_Izz}" link_com_origin="${link_4_com_xyz}" link_com_rpy="${link_4_com_rpy}"/>
-		<xacro:jaco_joint joint_name="${joint_4}" type="revolute" parent="${link_3}" child="${link}_4" joint_axis_xyz="${joint_4_axis_xyz}" joint_origin_xyz="${joint_4_origin_xyz}" joint_origin_rpy="${joint_4_origin_rpy}" lower_limit="-${J_LIM}" upper_limit="${J_LIM}"  />
+		<xacro:jaco_joint joint_name="${joint_4}" type="revolute" parent="${link_3}" child="${link}_4" joint_axis_xyz="${joint_4_axis_xyz}" joint_origin_xyz="${joint_4_origin_xyz}" joint_origin_rpy="${joint_4_origin_rpy}" lower_limit="${joint_4_lower_limit}" upper_limit="${joint_4_upper_limit}"  />
         <xacro:jaco_transmission joint_name="${joint_4}" />
 		<xacro:jaco_link_4_5 link_name="${link}" suffix="5" link_mass="${link_5_mass}" Ixx="${link_5_Ixx}" Ixy="${link_5_Ixy}" Ixz="${link_5_Ixz}" Iyy="${link_5_Iyy}" Iyz="${link_5_Iyz}" Izz="${link_5_Izz}" link_com_origin="${link_5_com_xyz}" link_com_rpy="${link_5_com_rpy}"/>
-		<xacro:jaco_joint joint_name="${joint_5}" type="revolute" parent="${link}_4" child="${link}_5" joint_axis_xyz="${joint_5_axis_xyz}" joint_origin_xyz="${joint_5_origin_xyz}" joint_origin_rpy="${joint_5_origin_rpy}" lower_limit="-${J_LIM}" upper_limit="${J_LIM}"/>
+		<xacro:jaco_joint joint_name="${joint_5}" type="revolute" parent="${link}_4" child="${link}_5" joint_axis_xyz="${joint_5_axis_xyz}" joint_origin_xyz="${joint_5_origin_xyz}" joint_origin_rpy="${joint_5_origin_rpy}" lower_limit="${joint_5_lower_limit}" upper_limit="${joint_5_upper_limit}"/>
         <xacro:jaco_transmission joint_name="${joint_5}" />
 		<xacro:jaco_link link_name="${link_hand}" link_mass="${link_hand_mass}" Ixx="${link_hand_Ixx}" Ixy="${link_hand_Ixy}" Ixz="${link_hand_Ixz}" Iyy="${link_hand_Iyy}" Iyz="${link_hand_Iyz}" Izz="${link_hand_Izz}" link_com_origin="${link_hand_com_xyz}" link_com_rpy="${link_hand_com_rpy}"/>
-		<xacro:jaco_joint joint_name="${joint_6}" type="revolute" parent="${link}_5" child="${link_hand}" joint_axis_xyz="${joint_6_axis_xyz}" joint_origin_xyz="${joint_6_origin_xyz}" joint_origin_rpy="${joint_6_origin_rpy}" lower_limit="-${J_LIM}" upper_limit="${J_LIM}"/>
+		<xacro:jaco_joint joint_name="${joint_6}" type="revolute" parent="${link}_5" child="${link_hand}" joint_axis_xyz="${joint_6_axis_xyz}" joint_origin_xyz="${joint_6_origin_xyz}" joint_origin_rpy="${joint_6_origin_rpy}" lower_limit="${joint_6_lower_limit}" upper_limit="${joint_6_upper_limit}"/>
         <xacro:jaco_transmission joint_name="${joint_6}" />
 		<xacro:jaco_ring_cover suffix="1" size="large"/>

Commit message: Improve moveit config

File: jaco2_description/urdf/jaco_arm.urdf.xacro (robot description, xacro)
@@ -178,5 +178,5 @@
 			<collision>
 				<geometry>
-					<mesh scale="${M_SCALE} ${M_SCALE} ${M_SCALE}" filename="package://jaco2_description/meshes/${link_name}.stl" />
+					<mesh scale="${M_SCALE} ${M_SCALE} ${M_SCALE}" filename="package://jaco2_description/meshes/${link_name}_potato.stl" />
 				</geometry>
 			</collision>
@@ -222,5 +222,5 @@
 			<collision>
 				<geometry>
-					<mesh scale="${M_SCALE} ${M_SCALE} ${M_SCALE}" filename="package://jaco2_description/meshes/${link_name}_4_5.stl" />
+					<mesh scale="${M_SCALE} ${M_SCALE} ${M_SCALE}" filename="package://jaco2_description/meshes/${link_name}_4_5_potato.stl" />
 				</geometry>
 			</collision>

File: jaco2_description/urdf/jaco_arm_with_realsense.urdf.xacro (robot description, xacro)
@@ -178,5 +178,5 @@
 			<collision>
 				<geometry>
-					<mesh scale="${M_SCALE} ${M_SCALE} ${M_SCALE}" filename="package://jaco2_description/meshes/${link_name}.stl" />
+					<mesh scale="${M_SCALE} ${M_SCALE} ${M_SCALE}" filename="package://jaco2_description/meshes/${link_name}_potato.stl" />
 				</geometry>
 			</collision>
@@ -200,5 +200,5 @@
 			<collision>
 				<geometry>
-					<mesh scale="${M_SCALE} ${M_SCALE} ${M_SCALE}" filename="package://jaco2_description/meshes/${file}.stl" />
+					<mesh scale="${M_SCALE} ${M_SCALE} ${M_SCALE}" filename="package://jaco2_description/meshes/${file}_convex_hull.stl" />
 				</geometry>
 			</collision>
@@ -244,5 +244,5 @@
 			<collision>
 				<geometry>
-					<mesh scale="${M_SCALE} ${M_SCALE} ${M_SCALE}" filename="package://jaco2_description/meshes/${link_name}_4_5.stl" />
+					<mesh scale="${M_SCALE} ${M_SCALE} ${M_SCALE}" filename="package://jaco2_description/meshes/${link_name}_4_5_potato.stl" />
 				</geometry>
 			</collision>

Commit message: Update collada files

File: jaco2_description/urdf/jaco_arm.urdf.xacro (robot description, xacro)
@@ -13,5 +13,6 @@
 	xmlns:physics="http://playerstage.sourceforge.net/gazebo/xmlschema/#physics"
 	xmlns:xacro="http://ros.org/wiki/xacro">
-    <xacro:property name="M_SCALE" value="0.0254" />
+        <xacro:property name="M_SCALE" value="0.0254" />
+        <xacro:property name="M_SCALE_1" value="1.0" />
 	<xacro:property name="M_PI" value="3.1415926535897931" />
 	<xacro:property name="J_LIM" value="${2*M_PI}" />
@@ -64,18 +65,18 @@
   <xacro:property name="joint_finger_1" value="jaco_joint_finger_1" />
   <xacro:property name="joint_finger_1_axis_xyz" value="0 0 1" />
-  <xacro:property name="joint_finger_1_origin_xyz" value="-0.032578 0.0033 -0.12131" />
-  <xacro:property name="joint_finger_1_origin_rpy" value="-1.7983 1.117 3.1416" />
+  <xacro:property name="joint_finger_1_origin_xyz" value="-0.03126 0.00279 -0.11467" />
+  <xacro:property name="joint_finger_1_origin_rpy" value="-1.7983 1.05 3.1416" />
   <xacro:property name="joint_finger_1_lower_limit" value="0" />
   <xacro:property name="joint_finger_1_upper_limit" value="${M_PI/180*40}" />
   <xacro:property name="joint_finger_3" value="jaco_joint_finger_3" />
   <xacro:property name="joint_finger_3_axis_xyz" value="0 0 1" />
-  <xacro:property name="joint_finger_3_origin_xyz" value="0.027788 -0.0206 -0.12131" />
-  <xacro:property name="joint_finger_3_origin_rpy" value="-1.6222 1.117 -0.23615" />
+  <xacro:property name="joint_finger_3_origin_xyz" value="0.02707 -0.0226 -0.11482" />
+  <xacro:property name="joint_finger_3_origin_rpy" value="-1.6222 1.05 -0.23615" />
   <xacro:property name="joint_finger_3_lower_limit" value="0" />
   <xacro:property name="joint_finger_3_upper_limit" value="${M_PI/180*40}" />
   <xacro:property name="joint_finger_2" value="jaco_joint_finger_2" />
   <xacro:property name="joint_finger_2_axis_xyz" value="0 0 1" />
-  <xacro:property name="joint_finger_2_origin_xyz" value="0.027788 0.0206 -0.12131" />
-  <xacro:property name="joint_finger_2_origin_rpy" value="-1.5161 1.1459 0.23978" />
+  <xacro:property name="joint_finger_2_origin_xyz" value="0.02707 0.0226 -0.11482" />
+  <xacro:property name="joint_finger_2_origin_rpy" value="-1.5161 1.05 0.23978" />
   <xacro:property name="joint_finger_2_lower_limit" value="0" />
   <xacro:property name="joint_finger_2_upper_limit" value="${M_PI/180*40}" />
@@ -170,5 +171,5 @@
 			<visual>
 				<geometry>
-					<mesh scale="${M_SCALE} ${M_SCALE} ${M_SCALE}" filename="package://jaco2_description/meshes/${link_name}.min.dae" />
+					<mesh scale="${M_SCALE_1} ${M_SCALE_1} ${M_SCALE_1}" filename="package://jaco2_description/meshes/${link_name}.min.dae" />
 				</geometry>
 				<material name="carbon_fiber">
@@ -192,5 +193,5 @@
 			<visual>
 				<geometry>
-					<mesh scale="${M_SCALE} ${M_SCALE} ${M_SCALE}" filename="package://jaco2_description/meshes/${link_name}.min.dae" />
+					<mesh scale="${M_SCALE_1} ${M_SCALE_1} ${M_SCALE_1}" filename="package://jaco2_description/meshes/${link_name}.min.dae" />
 				</geometry>
 				<material name="carbon_fiber">
@@ -214,5 +215,5 @@
 			<visual>
 				<geometry>
-					<mesh scale="${M_SCALE} ${M_SCALE} ${M_SCALE}" filename="package://jaco2_description/meshes/${link_name}_4_5.min.dae" />
+					<mesh scale="${M_SCALE_1} ${M_SCALE_1} ${M_SCALE_1}" filename="package://jaco2_description/meshes/${link_name}_4_5.min.dae" />
 				</geometry>
 				<material name="carbon_fiber">
