Commit message: Update Jaco2 model

File: jaco2_description/urdf/jaco_arm.urdf.xacro (robot description, xacro)
@@ -179,5 +179,5 @@
 			<collision>
 				<geometry>
-					<mesh scale="${M_SCALE} ${M_SCALE} ${M_SCALE}" filename="package://jaco2_description/meshes/${link_name}_potato.stl" />
+					<mesh scale="${M_SCALE_1} ${M_SCALE_1} ${M_SCALE_1}" filename="package://jaco2_description/meshes/${link_name}_potato.stl" />
 				</geometry>
 			</collision>
@@ -187,6 +187,6 @@
 		<link name="${link_name}_${suffix}">
             <inertial>
-                <mass value="0.25"/>
-                <inertia ixx="0.01" ixy="0" ixz="0" iyy="0.01" iyz="0" izz="0.01"/>
+                <mass value="0.0"/>
+                <inertia ixx="0.0" ixy="0" ixz="0" iyy="0.0" iyz="0" izz="0.0"/>
                 <origin/>
             </inertial>
@@ -201,5 +201,5 @@
 			<collision>
 				<geometry>
-					<mesh scale="${M_SCALE} ${M_SCALE} ${M_SCALE}" filename="package://jaco2_description/meshes/${link_name}.stl" />
+					<mesh scale="${M_SCALE_1} ${M_SCALE_1} ${M_SCALE_1}" filename="package://jaco2_description/meshes/${link_name}.stl" />
 				</geometry>
 			</collision>
@@ -223,5 +223,5 @@
 			<collision>
 				<geometry>
-					<mesh scale="${M_SCALE} ${M_SCALE} ${M_SCALE}" filename="package://jaco2_description/meshes/${link_name}_4_5_potato.stl" />
+					<mesh scale="${M_SCALE_1} ${M_SCALE_1} ${M_SCALE_1}" filename="package://jaco2_description/meshes/${link_name}_4_5_potato.stl" />
 				</geometry>
 			</collision>

File: jaco2_description/urdf/jaco_arm_left.urdf.xacro (robot description, xacro)
@@ -13,5 +13,6 @@
 	xmlns:physics="http://playerstage.sourceforge.net/gazebo/xmlschema/#physics"
 	xmlns:xacro="http://ros.org/wiki/xacro">
-    <xacro:property name="M_SCALE" value="0.0254" />
+        <xacro:property name="M_SCALE" value="0.0254" />
+        <xacro:property name="M_SCALE_1" value="1.0" />
 	<xacro:property name="M_PI" value="3.1415926535897931" />
 	<xacro:property name="J_LIM" value="${2*M_PI}" />
@@ -37,42 +38,52 @@
   <xacro:property name="joint_1" value="jaco_left_joint_1" />
   <xacro:property name="joint_1_axis_xyz" value="0 0 1" />
-  <xacro:property name="joint_1_origin_xyz" value="0 0 0.1535" />
+  <xacro:property name="joint_1_origin_xyz" value="0 0 0.15675" />
   <xacro:property name="joint_1_origin_rpy" value="${M_PI} 0 0" />
   <xacro:property name="joint_2" value="jaco_left_joint_2" />
   <xacro:property name="joint_2_axis_xyz" value="0 0 1" />
-  <xacro:property name="joint_2_origin_xyz" value="0 0 -0.1185" />
+  <xacro:property name="joint_2_origin_xyz" value="0 0.0016 -0.11875" />
   <xacro:property name="joint_2_origin_rpy" value="-${M_PI/2} -${M_PI/2} 0" />
+  <xacro:property name="joint_2_lower_limit" value="${M_PI/180*50}" />
+  <xacro:property name="joint_2_upper_limit" value="${M_PI/180*310}" />
   <xacro:property name="joint_3" value="jaco_left_joint_3" />
   <xacro:property name="joint_3_axis_xyz" value="0 0 1" />
   <xacro:property name="joint_3_origin_xyz" value="0.41 0 0" />
   <xacro:property name="joint_3_origin_rpy" value="${M_PI} 0 ${M_PI}" />
+  <xacro:property name="joint_3_lower_limit" value="${M_PI/180*19}" />
+  <xacro:property name="joint_3_upper_limit" value="${M_PI/180*341}" />
   <xacro:property name="joint_4" value="jaco_left_joint_4" />
   <xacro:property name="joint_4_axis_xyz" value="0 0 1" />
-  <xacro:property name="joint_4_origin_xyz" value="0.207 0 -0.01125" />
+  <xacro:property name="joint_4_origin_xyz" value="0.2073 0 -0.0114" />
   <xacro:property name="joint_4_origin_rpy" value="0 -${M_PI/2} 0" />
+  <xacro:property name="joint_4_lower_limit" value="${-2*M_PI}" />
+  <xacro:property name="joint_4_upper_limit" value="${2*M_PI}" />
   <xacro:property name="joint_5" value="jaco_left_joint_5" />
   <xacro:property name="joint_5_axis_xyz" value="0 0 1" />
   <xacro:property name="joint_5_origin_xyz" value="0.03705 0 -0.0641725" />
   <xacro:property name="joint_5_origin_rpy" value="0 ${M_PI/180*60} ${M_PI}" /> <!-- maybe 55 degrees, Advanded user guide specifys 60 ...-->
+  <xacro:property name="joint_5_lower_limit" value="${-2*M_PI}" />
+  <xacro:property name="joint_5_upper_limit" value="${2*M_PI}" />
   <xacro:property name="joint_6" value="jaco_left_joint_6" />
   <xacro:property name="joint_6_axis_xyz" value="0 0 1" />
   <xacro:property name="joint_6_origin_xyz" value="0.03705 0 -0.0641725" />
   <xacro:property name="joint_6_origin_rpy" value="0 ${M_PI/180*60} ${M_PI}" /> <!-- maybe 55 degrees, Advanded user guide specifys 60 ...-->
+  <xacro:property name="joint_6_lower_limit" value="${-2*M_PI}" />
+  <xacro:property name="joint_6_upper_limit" value="${2*M_PI}" />
   <xacro:property name="joint_finger_1" value="jaco_left_joint_finger_1" />
   <xacro:property name="joint_finger_1_axis_xyz" value="0 0 1" />
-  <xacro:property name="joint_finger_1_origin_xyz" value="-0.032578 0.0033 -0.12131" />
-  <xacro:property name="joint_finger_1_origin_rpy" value="-1.7983 1.117 3.1416" />
+  <xacro:property name="joint_finger_1_origin_xyz" value="-0.03126 0.00279 -0.11467" />
+  <xacro:property name="joint_finger_1_origin_rpy" value="-1.7983 1.05 3.1416" />
   <xacro:property name="joint_finger_1_lower_limit" value="0" />
   <xacro:property name="joint_finger_1_upper_limit" value="${M_PI/180*40}" />
   <xacro:property name="joint_finger_3" value="jaco_left_joint_finger_3" />
   <xacro:property name="joint_finger_3_axis_xyz" value="0 0 1" />
-  <xacro:property name="joint_finger_3_origin_xyz" value="0.027788 -0.0206 -0.12131" />
-  <xacro:property name="joint_finger_3_origin_rpy" value="-1.6222 1.117 -0.23615" />
+  <xacro:property name="joint_finger_3_origin_xyz" value="0.02707 -0.0226 -0.11482" />
+  <xacro:property name="joint_finger_3_origin_rpy" value="-1.6222 1.05 -0.23615" />
   <xacro:property name="joint_finger_3_lower_limit" value="0" />
   <xacro:property name="joint_finger_3_upper_limit" value="${M_PI/180*40}" />
   <xacro:property name="joint_finger_2" value="jaco_left_joint_finger_2" />
   <xacro:property name="joint_finger_2_axis_xyz" value="0 0 1" />
-  <xacro:property name="joint_finger_2_origin_xyz" value="0.027788 0.0206 -0.12131" />
-  <xacro:property name="joint_finger_2_origin_rpy" value="-1.5161 1.1459 0.23978" />
+  <xacro:property name="joint_finger_2_origin_xyz" value="0.02707 0.0226 -0.11482" />
+  <xacro:property name="joint_finger_2_origin_rpy" value="-1.5161 1.05 0.23978" />
   <xacro:property name="joint_finger_2_lower_limit" value="0" />
   <xacro:property name="joint_finger_2_upper_limit" value="${M_PI/180*40}" />
@@ -167,5 +178,5 @@
 			<visual>
 				<geometry>
-					<mesh scale="${M_SCALE} ${M_SCALE} ${M_SCALE}" filename="package://jaco2_description/meshes/${mesh_name}.min.dae" />
+					<mesh scale="${M_SCALE_1} ${M_SCALE_1} ${M_SCALE_1}" filename="package://jaco2_description/meshes/${link_name}.min.dae" />
 				</geometry>
 				<material name="carbon_fiber">
@@ -175,5 +186,5 @@
 			<collision>
 				<geometry>
-					<mesh scale="${M_SCALE} ${M_SCALE} ${M_SCALE}" filename="package://jaco2_description/meshes/${mesh_name}.stl" />
+					<mesh scale="${M_SCALE_1} ${M_SCALE_1} ${M_SCALE_1}" filename="package://jaco2_description/meshes/${link_name}_potato.stl" />
 				</geometry>
 			</collision>
@@ -189,5 +200,5 @@
 			<visual>
 				<geometry>
-					<mesh scale="${M_SCALE} ${M_SCALE} ${M_SCALE}" filename="package://jaco2_description/meshes//${mesh_name}.min.dae" />
+					<mesh scale="${M_SCALE_1} ${M_SCALE_1} ${M_SCALE_1}" filename="package://jaco2_description/meshes/${link_name}.min.dae" />
 				</geometry>
 				<material name="carbon_fiber">
@@ -197,5 +208,5 @@
 			<collision>
 				<geometry>
-					<mesh scale="${M_SCALE} ${M_SCALE} ${M_SCALE}" filename="package://jaco2_description/meshes//${mesh_name}.stl" />
+					<mesh scale="${M_SCALE_1} ${M_SCALE_1} ${M_SCALE_1}" filename="package://jaco2_description/meshes/${link_name}.stl" />
 				</geometry>
 			</collision>
@@ -211,5 +222,5 @@
 			<visual>
 				<geometry>
-					<mesh scale="${M_SCALE} ${M_SCALE} ${M_SCALE}" filename="package://jaco2_description/meshes//${mesh_name}_4_5.min.dae" />
+					<mesh scale="${M_SCALE_1} ${M_SCALE_1} ${M_SCALE_1}" filename="package://jaco2_description/meshes/${link_name}_4_5.min.dae" />
 				</geometry>
 				<material name="carbon_fiber">
@@ -219,5 +230,5 @@
 			<collision>
 				<geometry>
-					<mesh scale="${M_SCALE} ${M_SCALE} ${M_SCALE}" filename="package://jaco2_description/meshes//${mesh_name}_4_5.stl" />
+					<mesh scale="${M_SCALE_1} ${M_SCALE_1} ${M_SCALE_1}" filename="package://jaco2_description/meshes/${link_name}_4_5_potato.stl" />
 				</geometry>
 			</collision>

File: jaco2_description/urdf/jaco_arm_right.urdf.xacro (robot description, xacro)
@@ -13,17 +13,18 @@
 	xmlns:physics="http://playerstage.sourceforge.net/gazebo/xmlschema/#physics"
 	xmlns:xacro="http://ros.org/wiki/xacro">
-    <xacro:property name="M_SCALE" value="0.0254" />
-	<xacro:property name="M_PI" value="3.1415926535897931" />
-	<xacro:property name="J_LIM" value="${2*M_PI}" />
-	<xacro:property name="link_base" value="jaco_right_link_base" />
-	<xacro:property name="link" value="jaco_right_link" />
-	<xacro:property name="link_1" value="jaco_right_link_1" />
-	<xacro:property name="link_2" value="jaco_right_link_2" />
-	<xacro:property name="link_3" value="jaco_right_link_3" />
-	<xacro:property name="link_hand" value="jaco_right_link_hand" />
-	<xacro:property name="link_finger" value="jaco_right_link_finger" />
-	<xacro:property name="link_finger_tip" value="jaco_right_link_finger_tip" />
-	<xacro:property name="joint_base" value="jaco_right_joint_base" />
-	<xacro:property name="joint_base_axis_xyz" value="0 0 0" />
+  <xacro:property name="M_SCALE" value="0.0254" />
+  <xacro:property name="M_SCALE_1" value="1.0" />
+  <xacro:property name="M_PI" value="3.1415926535897931" />
+  <xacro:property name="J_LIM" value="${2*M_PI}" />
+  <xacro:property name="link_base" value="jaco_right_link_base" />
+  <xacro:property name="link" value="jaco_right_link" />
+  <xacro:property name="link_1" value="jaco_right_link_1" />
+  <xacro:property name="link_2" value="jaco_right_link_2" />
+  <xacro:property name="link_3" value="jaco_right_link_3" />
+  <xacro:property name="link_hand" value="jaco_right_link_hand" />
+  <xacro:property name="link_finger" value="jaco_right_link_finger" />
+  <xacro:property name="link_finger_tip" value="jaco_right_link_finger_tip" />
+  <xacro:property name="joint_base" value="jaco_right_joint_base" />
+  <xacro:property name="joint_base_axis_xyz" value="0 0 0" />
   <xacro:property name="mesh_link_base" value="jaco_link_base" />
   <xacro:property name="mesh_link" value="jaco_link" />
@@ -36,42 +37,54 @@
   <xacro:property name="joint_1" value="jaco_right_joint_1" />
   <xacro:property name="joint_1_axis_xyz" value="0 0 1" />
-  <xacro:property name="joint_1_origin_xyz" value="0 0 0.1535" />
+  <xacro:property name="joint_1_origin_xyz" value="0 0 0.15675" />
   <xacro:property name="joint_1_origin_rpy" value="${M_PI} 0 0" />
+  <xacro:property name="joint_1_lower_limit" value="${-2*M_PI}" />
+  <xacro:property name="joint_1_upper_limit" value="${2*M_PI}" />
   <xacro:property name="joint_2" value="jaco_right_joint_2" />
   <xacro:property name="joint_2_axis_xyz" value="0 0 1" />
-  <xacro:property name="joint_2_origin_xyz" value="0 0 -0.1185" />
+  <xacro:property name="joint_2_origin_xyz" value="0 0.0016 -0.11875" />
   <xacro:property name="joint_2_origin_rpy" value="-${M_PI/2} -${M_PI/2} 0" />
+  <xacro:property name="joint_2_lower_limit" value="${M_PI/180*50}" />
+  <xacro:property name="joint_2_upper_limit" value="${M_PI/180*310}" />
   <xacro:property name="joint_3" value="jaco_right_joint_3" />
   <xacro:property name="joint_3_axis_xyz" value="0 0 1" />
   <xacro:property name="joint_3_origin_xyz" value="0.41 0 0" />
   <xacro:property name="joint_3_origin_rpy" value="${M_PI} 0 ${M_PI}" />
+  <xacro:property name="joint_3_lower_limit" value="${M_PI/180*19}" />
+  <xacro:property name="joint_3_upper_limit" value="${M_PI/180*341}" />
   <xacro:property name="joint_4" value="jaco_right_joint_4" />
   <xacro:property name="joint_4_axis_xyz" value="0 0 1" />
-  <xacro:property name="joint_4_origin_xyz" value="0.207 0 -0.01125" />
+  <xacro:property name="joint_4_origin_xyz" value="0.2073 0 -0.0114" />
   <xacro:property name="joint_4_origin_rpy" value="0 -${M_PI/2} 0" />
+  <xacro:property name="joint_4_lower_limit" value="${-2*M_PI}" />
+  <xacro:property name="joint_4_upper_limit" value="${2*M_PI}" />
   <xacro:property name="joint_5" value="jaco_right_joint_5" />
   <xacro:property name="joint_5_axis_xyz" value="0 0 1" />
   <xacro:property name="joint_5_origin_xyz" value="0.03705 0 -0.0641725" />
   <xacro:property name="joint_5_origin_rpy" value="0 ${M_PI/180*60} ${M_PI}" /> <!-- maybe 55 degrees, Advanded user guide specifys 60 ...-->
+  <xacro:property name="joint_5_lower_limit" value="${-2*M_PI}" />
+  <xacro:property name="joint_5_upper_limit" value="${2*M_PI}" />
   <xacro:property name="joint_6" value="jaco_right_joint_6" />
   <xacro:property name="joint_6_axis_xyz" value="0 0 1" />
   <xacro:property name="joint_6_origin_xyz" value="0.03705 0 -0.0641725" />
   <xacro:property name="joint_6_origin_rpy" value="0 ${M_PI/180*60} ${M_PI}" /> <!-- maybe 55 degrees, Advanded user guide specifys 60 ...-->
+  <xacro:property name="joint_6_lower_limit" value="${-2*M_PI}" />
+  <xacro:property name="joint_6_upper_limit" value="${2*M_PI}" />
   <xacro:property name="joint_finger_1" value="jaco_right_joint_finger_1" />
   <xacro:property name="joint_finger_1_axis_xyz" value="0 0 1" />
-  <xacro:property name="joint_finger_1_origin_xyz" value="-0.032578 0.0033 -0.12131" />
-  <xacro:property name="joint_finger_1_origin_rpy" value="-1.7983 1.117 3.1416" />
+  <xacro:property name="joint_finger_1_origin_xyz" value="-0.03126 0.00279 -0.11467" />
+  <xacro:property name="joint_finger_1_origin_rpy" value="-1.7983 1.05 3.1416" />
   <xacro:property name="joint_finger_1_lower_limit" value="0" />
   <xacro:property name="joint_finger_1_upper_limit" value="${M_PI/180*40}" />
   <xacro:property name="joint_finger_3" value="jaco_right_joint_finger_3" />
   <xacro:property name="joint_finger_3_axis_xyz" value="0 0 1" />
-  <xacro:property name="joint_finger_3_origin_xyz" value="0.027788 -0.0206 -0.12131" />
-  <xacro:property name="joint_finger_3_origin_rpy" value="-1.6222 1.117 -0.23615" />
+  <xacro:property name="joint_finger_3_origin_xyz" value="0.02707 -0.0226 -0.11482" />
+  <xacro:property name="joint_finger_3_origin_rpy" value="-1.6222 1.05 -0.23615" />
   <xacro:property name="joint_finger_3_lower_limit" value="0" />
   <xacro:property name="joint_finger_3_upper_limit" value="${M_PI/180*40}" />
   <xacro:property name="joint_finger_2" value="jaco_right_joint_finger_2" />
   <xacro:property name="joint_finger_2_axis_xyz" value="0 0 1" />
-  <xacro:property name="joint_finger_2_origin_xyz" value="0.027788 0.0206 -0.12131" />
-  <xacro:property name="joint_finger_2_origin_rpy" value="-1.5161 1.1459 0.23978" />
+  <xacro:property name="joint_finger_2_origin_xyz" value="0.02707 0.0226 -0.11482" />
+  <xacro:property name="joint_finger_2_origin_rpy" value="-1.5161 1.05 0.23978" />
   <xacro:property name="joint_finger_2_lower_limit" value="0" />
   <xacro:property name="joint_finger_2_upper_limit" value="${M_PI/180*40}" />
@@ -166,5 +179,5 @@
 			<visual>
 				<geometry>
-					<mesh scale="${M_SCALE} ${M_SCALE} ${M_SCALE}" filename="package://jaco2_description/meshes//${mesh_name}.min.dae" />
+					<mesh scale="${M_SCALE_1} ${M_SCALE_1} ${M_SCALE_1}" filename="package://jaco2_description/meshes/${link_name}.min.dae" />
 				</geometry>
 				<material name="carbon_fiber">
@@ -174,5 +187,5 @@
 			<collision>
 				<geometry>
-					<mesh scale="${M_SCALE} ${M_SCALE} ${M_SCALE}" filename="package://jaco2_description/meshes//${mesh_name}.stl" />
+					<mesh scale="${M_SCALE_1} ${M_SCALE_1} ${M_SCALE_1}" filename="package://jaco2_description/meshes/${link_name}_potato.stl" />
 				</geometry>
 			</collision>
@@ -182,11 +195,11 @@
 		<link name="${link_name}_${suffix}">
             <inertial>
-                <mass value="0.25"/>
-                <inertia ixx="0.01" ixy="0" ixz="0" iyy="0.01" iyz="0" izz="0.01"/>
+                <mass value="0.0"/>
+                <inertia ixx="0.0" ixy="0" ixz="0" iyy="0.0" iyz="0" izz="0.0"/>
                 <origin/>
             </inertial>
 			<visual>
 				<geometry>
-					<mesh scale="${M_SCALE} ${M_SCALE} ${M_SCALE}" filename="package://jaco2_description/meshes//${mesh_name}.min.dae" />
+					<mesh scale="${M_SCALE_1} ${M_SCALE_1} ${M_SCALE_1}" filename="package://jaco2_description/meshes/${link_name}.min.dae" />
 				</geometry>
 				<material name="carbon_fiber">
@@ -196,5 +209,5 @@
 			<collision>
 				<geometry>
-					<mesh scale="${M_SCALE} ${M_SCALE} ${M_SCALE}" filename="package://jaco2_description/meshes//${mesh_name}.stl" />
+					<mesh scale="${M_SCALE_1} ${M_SCALE_1} ${M_SCALE_1}" filename="package://jaco2_description/meshes/${link_name}.stl" />
 				</geometry>
 			</collision>
@@ -210,5 +223,5 @@
 			<visual>
 				<geometry>
-					<mesh scale="${M_SCALE} ${M_SCALE} ${M_SCALE}" filename="package://jaco2_description/meshes//${mesh_name}_4_5.min.dae" />
+					<mesh scale="${M_SCALE_1} ${M_SCALE_1} ${M_SCALE_1}" filename="package://jaco2_description/meshes/${link_name}_4_5.min.dae" />
 				</geometry>
 				<material name="carbon_fiber">
@@ -218,5 +231,5 @@
 			<collision>
 				<geometry>
-					<mesh scale="${M_SCALE} ${M_SCALE} ${M_SCALE}" filename="package://jaco2_description/meshes//${mesh_name}_4_5.stl" />
+					<mesh scale="${M_SCALE_1} ${M_SCALE_1} ${M_SCALE_1}" filename="package://jaco2_description/meshes/${link_name}_4_5_potato.stl" />
 				</geometry>
 			</collision>
