Commit message: Update Jaco2 model

File: jaco2_description/urdf/jaco_arm_with_realsense.urdf.xacro (robot description, xacro)
@@ -13,23 +13,24 @@
 	xmlns:physics="http://playerstage.sourceforge.net/gazebo/xmlschema/#physics"
 	xmlns:xacro="http://ros.org/wiki/xacro">
-    <xacro:property name="M_SCALE" value="0.0254" />
-	<xacro:property name="M_PI" value="3.1415926535897931" />
-	<xacro:property name="J_LIM" value="${2*M_PI}" />
-	<xacro:property name="link_base" value="jaco_link_base" />
-	<xacro:property name="link" value="jaco_link" />
-	<xacro:property name="link_1" value="jaco_link_1" />
-	<xacro:property name="link_2" value="jaco_link_2" />
-	<xacro:property name="link_3" value="jaco_link_3" />
-	<xacro:property name="link_hand" value="jaco_link_hand" />
-	<xacro:property name="link_finger" value="jaco_link_finger" />
-	<xacro:property name="link_finger_tip" value="jaco_link_finger_tip" />
-	<xacro:property name="joint_base" value="jaco_joint_base" />
-	<xacro:property name="joint_base_axis_xyz" value="0 0 0" />
+  <xacro:property name="M_SCALE" value="0.0254" />
+  <xacro:property name="M_SCALE_1" value="1.0" />
+  <xacro:property name="M_PI" value="3.1415926535897931" />
+  <xacro:property name="J_LIM" value="${2*M_PI}" />
+  <xacro:property name="link_base" value="jaco_link_base" />
+  <xacro:property name="link" value="jaco_link" />
+  <xacro:property name="link_1" value="jaco_link_1" />
+  <xacro:property name="link_2" value="jaco_link_2" />
+  <xacro:property name="link_3" value="jaco_link_3" />
+  <xacro:property name="link_hand" value="jaco_link_hand" />
+  <xacro:property name="link_finger" value="jaco_link_finger" />
+  <xacro:property name="link_finger_tip" value="jaco_link_finger_tip" />
+  <xacro:property name="joint_base" value="jaco_joint_base" />
+  <xacro:property name="joint_base_axis_xyz" value="0 0 0" />
   <xacro:property name="joint_1" value="jaco_joint_1" />
   <xacro:property name="joint_1_axis_xyz" value="0 0 1" />
   <xacro:property name="joint_1_origin_xyz" value="0 0 0.15675" />
   <xacro:property name="joint_1_origin_rpy" value="${M_PI} 0 0" />
-  <xacro:property name="joint_1_lower_limit" value="${0.5*M_PI}" />
-  <xacro:property name="joint_1_upper_limit" value="${2.5*M_PI}" />
+  <xacro:property name="joint_1_lower_limit" value="${-M_PI-0.1}" />
+  <xacro:property name="joint_1_upper_limit" value="${M_PI+0.1}" />
   <xacro:property name="joint_2" value="jaco_joint_2" />
   <xacro:property name="joint_2_axis_xyz" value="0 0 1" />
@@ -48,34 +49,34 @@
   <xacro:property name="joint_4_origin_xyz" value="0.2073 0 -0.0114" />
   <xacro:property name="joint_4_origin_rpy" value="0 -${M_PI/2} 0" />
-  <xacro:property name="joint_4_lower_limit" value="${0.5*M_PI}" />
-  <xacro:property name="joint_4_upper_limit" value="${2.5*M_PI}" />
+  <xacro:property name="joint_4_lower_limit" value="${-M_PI-0.1}" />
+  <xacro:property name="joint_4_upper_limit" value="${M_PI+0.1}" />
   <xacro:property name="joint_5" value="jaco_joint_5" />
   <xacro:property name="joint_5_axis_xyz" value="0 0 1" />
   <xacro:property name="joint_5_origin_xyz" value="0.03705 0 -0.0641725" />
-  <xacro:property name="joint_5_origin_rpy" value="0 ${M_PI/180*60} ${M_PI}" /> <!-- maybe 55 degrees, Advanded user guide specifys 60 ...-->
-  <xacro:property name="joint_5_lower_limit" value="${-M_PI}" />
-  <xacro:property name="joint_5_upper_limit" value="${M_PI}" />
+  <xacro:property name="joint_5_origin_rpy" value="0 ${M_PI/180*60} ${M_PI}" />
+  <xacro:property name="joint_5_lower_limit" value="${-M_PI-0.1}" />
+  <xacro:property name="joint_5_upper_limit" value="${M_PI+0.1}" />
   <xacro:property name="joint_6" value="jaco_joint_6" />
   <xacro:property name="joint_6_axis_xyz" value="0 0 1" />
   <xacro:property name="joint_6_origin_xyz" value="0.03705 0 -0.0641725" />
-  <xacro:property name="joint_6_origin_rpy" value="0 ${M_PI/180*60} ${M_PI}" /> <!-- maybe 55 degrees, Advanded user guide specifys 60 ...-->
-  <xacro:property name="joint_6_lower_limit" value="${-M_PI}" />
-  <xacro:property name="joint_6_upper_limit" value="${M_PI}" />
+  <xacro:property name="joint_6_origin_rpy" value="0 ${M_PI/180*60} ${M_PI}" />
+  <xacro:property name="joint_6_lower_limit" value="${-M_PI-0.1}" />
+  <xacro:property name="joint_6_upper_limit" value="${M_PI+0.1}" />
   <xacro:property name="joint_finger_1" value="jaco_joint_finger_1" />
   <xacro:property name="joint_finger_1_axis_xyz" value="0 0 1" />
-  <xacro:property name="joint_finger_1_origin_xyz" value="-0.032578 0.0033 -0.12131" />
-  <xacro:property name="joint_finger_1_origin_rpy" value="-1.7983 1.117 3.1416" />
+  <xacro:property name="joint_finger_1_origin_xyz" value="-0.03126 0.00279 -0.11467" />
+  <xacro:property name="joint_finger_1_origin_rpy" value="-1.7983 1.05 3.1416" />
   <xacro:property name="joint_finger_1_lower_limit" value="0" />
   <xacro:property name="joint_finger_1_upper_limit" value="${M_PI/180*40}" />
   <xacro:property name="joint_finger_3" value="jaco_joint_finger_3" />
   <xacro:property name="joint_finger_3_axis_xyz" value="0 0 1" />
-  <xacro:property name="joint_finger_3_origin_xyz" value="0.027788 -0.0206 -0.12131" />
-  <xacro:property name="joint_finger_3_origin_rpy" value="-1.6222 1.117 -0.23615" />
+  <xacro:property name="joint_finger_3_origin_xyz" value="0.02707 -0.0226 -0.11482" />
+  <xacro:property name="joint_finger_3_origin_rpy" value="-1.6222 1.05 -0.23615" />
   <xacro:property name="joint_finger_3_lower_limit" value="0" />
   <xacro:property name="joint_finger_3_upper_limit" value="${M_PI/180*40}" />
   <xacro:property name="joint_finger_2" value="jaco_joint_finger_2" />
   <xacro:property name="joint_finger_2_axis_xyz" value="0 0 1" />
-  <xacro:property name="joint_finger_2_origin_xyz" value="0.027788 0.0206 -0.12131" />
-  <xacro:property name="joint_finger_2_origin_rpy" value="-1.5161 1.1459 0.23978" />
+  <xacro:property name="joint_finger_2_origin_xyz" value="0.02707 0.0226 -0.11482" />
+  <xacro:property name="joint_finger_2_origin_rpy" value="-1.5161 1.05 0.23978" />
   <xacro:property name="joint_finger_2_lower_limit" value="0" />
   <xacro:property name="joint_finger_2_upper_limit" value="${M_PI/180*40}" />
@@ -170,13 +171,13 @@
 			<visual>
 				<geometry>
-					<mesh scale="${M_SCALE} ${M_SCALE} ${M_SCALE}" filename="package://jaco2_description/meshes/${link_name}.min.dae" />
-				</geometry>
-				<material name="carbon_fiber">
-					<color rgba="0.792156862745098 0.819607843137255 0.933333333333333 1" />
-				</material>
-			</visual>
-			<collision>
-				<geometry>
-					<mesh scale="${M_SCALE} ${M_SCALE} ${M_SCALE}" filename="package://jaco2_description/meshes/${link_name}_potato.stl" />
+					<mesh scale="${M_SCALE_1} ${M_SCALE_1} ${M_SCALE_1}" filename="package://jaco2_description/meshes/${link_name}.min.dae" />
+				</geometry>
+				<material name="carbon_fiber">
+					<color rgba="0.792156862745098 0.819607843137255 0.933333333333333 1" />
+				</material>
+			</visual>
+			<collision>
+				<geometry>
+					<mesh scale="${M_SCALE_1} ${M_SCALE_1} ${M_SCALE_1}" filename="package://jaco2_description/meshes/${link_name}_potato.stl" />
 				</geometry>
 			</collision>
@@ -192,13 +193,13 @@
 			<visual>
 				<geometry>
-					<mesh scale="${M_SCALE} ${M_SCALE} ${M_SCALE}" filename="package://jaco2_description/meshes/${file}.dae" />
-				</geometry>
-				<material name="carbon_fiber">
-					<color rgba="0.792156862745098 0.819607843137255 0.933333333333333 1" />
-				</material>
-			</visual>
-			<collision>
-				<geometry>
-					<mesh scale="${M_SCALE} ${M_SCALE} ${M_SCALE}" filename="package://jaco2_description/meshes/${file}.stl" />
+					<mesh scale="${M_SCALE_1} ${M_SCALE_1} ${M_SCALE_1}" filename="package://jaco2_description/meshes/${file}.dae" />
+				</geometry>
+				<material name="carbon_fiber">
+					<color rgba="0.792156862745098 0.819607843137255 0.933333333333333 1" />
+				</material>
+			</visual>
+			<collision>
+				<geometry>
+					<mesh scale="${M_SCALE_1} ${M_SCALE_1} ${M_SCALE_1}" filename="package://jaco2_description/meshes/${file}.stl" />
 				</geometry>
 			</collision>
@@ -208,19 +209,19 @@
 		<link name="${link_name}_${suffix}">
             <inertial>
-                <mass value="0.25"/>
-                <inertia ixx="0.01" ixy="0" ixz="0" iyy="0.01" iyz="0" izz="0.01"/>
+                <mass value="0.0"/>
+                <inertia ixx="0.00" ixy="0" ixz="0" iyy="0.0" iyz="0" izz="0.0"/>
                 <origin/>
             </inertial>
 			<visual>
 				<geometry>
-					<mesh scale="${M_SCALE} ${M_SCALE} ${M_SCALE}" filename="package://jaco2_description/meshes/${link_name}.min.dae" />
-				</geometry>
-				<material name="carbon_fiber">
-					<color rgba="0.792156862745098 0.819607843137255 0.933333333333333 1" />
-				</material>
-			</visual>
-			<collision>
-				<geometry>
-					<mesh scale="${M_SCALE} ${M_SCALE} ${M_SCALE}" filename="package://jaco2_description/meshes/${link_name}.stl" />
+					<mesh scale="${M_SCALE_1} ${M_SCALE_1} ${M_SCALE_1}" filename="package://jaco2_description/meshes/${link_name}.min.dae" />
+				</geometry>
+				<material name="carbon_fiber">
+					<color rgba="0.792156862745098 0.819607843137255 0.933333333333333 1" />
+				</material>
+			</visual>
+			<collision>
+				<geometry>
+					<mesh scale="${M_SCALE_1} ${M_SCALE_1} ${M_SCALE_1}" filename="package://jaco2_description/meshes/${link_name}.stl" />
 				</geometry>
 			</collision>
@@ -236,13 +237,13 @@
 			<visual>
 				<geometry>
-					<mesh scale="${M_SCALE} ${M_SCALE} ${M_SCALE}" filename="package://jaco2_description/meshes/${link_name}_4_5.min.dae" />
-				</geometry>
-				<material name="carbon_fiber">
-					<color rgba="0.792156862745098 0.819607843137255 0.933333333333333 1" />
-				</material>
-			</visual>
-			<collision>
-				<geometry>
-					<mesh scale="${M_SCALE} ${M_SCALE} ${M_SCALE}" filename="package://jaco2_description/meshes/${link_name}_4_5_potato.stl" />
+					<mesh scale="${M_SCALE_1} ${M_SCALE_1} ${M_SCALE_1}" filename="package://jaco2_description/meshes/${link_name}_4_5.min.dae" />
+				</geometry>
+				<material name="carbon_fiber">
+					<color rgba="0.792156862745098 0.819607843137255 0.933333333333333 1" />
+				</material>
+			</visual>
+			<collision>
+				<geometry>
+					<mesh scale="${M_SCALE_1} ${M_SCALE_1} ${M_SCALE_1}" filename="package://jaco2_description/meshes/${link_name}_4_5_potato.stl" />
 				</geometry>
 			</collision>
@@ -324,5 +325,5 @@
 		<xacro:jaco_joint joint_name="${joint_5}" type="revolute" parent="${link}_4" child="${link}_5" joint_axis_xyz="${joint_5_axis_xyz}" joint_origin_xyz="${joint_5_origin_xyz}" joint_origin_rpy="${joint_5_origin_rpy}" lower_limit="${joint_5_lower_limit}" upper_limit="${joint_5_upper_limit}"/>
         <xacro:jaco_transmission joint_name="${joint_5}" />
-		<xacro:jaco_eeff_link link_name="${link_hand}" file="sick_hand_notloesung_inch" link_mass="${link_hand_mass}" Ixx="${link_hand_Ixx}" Ixy="${link_hand_Ixy}" Ixz="${link_hand_Ixz}" Iyy="${link_hand_Iyy}" Iyz="${link_hand_Iyz}" Izz="${link_hand_Izz}" link_com_origin="${link_hand_com_xyz}" link_com_rpy="${link_hand_com_rpy}"/>
+		<xacro:jaco_eeff_link link_name="${link_hand}" file="jaco_hand_with_realsense" link_mass="${link_hand_mass}" Ixx="${link_hand_Ixx}" Ixy="${link_hand_Ixy}" Ixz="${link_hand_Ixz}" Iyy="${link_hand_Iyy}" Iyz="${link_hand_Iyz}" Izz="${link_hand_Izz}" link_com_origin="${link_hand_com_xyz}" link_com_rpy="${link_hand_com_rpy}"/>
 		<xacro:jaco_joint joint_name="${joint_6}" type="revolute" parent="${link}_5" child="${link_hand}" joint_axis_xyz="${joint_6_axis_xyz}" joint_origin_xyz="${joint_6_origin_xyz}" joint_origin_rpy="${joint_6_origin_rpy}" lower_limit="${joint_6_lower_limit}" upper_limit="${joint_6_upper_limit}"/>
         <xacro:jaco_transmission joint_name="${joint_6}" />
@@ -337,6 +338,6 @@
 		<xacro:jaco_ring_cover suffix="2" size="small"/>
 		<xacro:jaco_joint joint_name="jaco_large_ring_cover_5_joint" type="fixed" parent="${link}_4" child="jaco_small_ring_cover_2" joint_axis_xyz="${joint_5_axis_xyz}" joint_origin_xyz="${joint_5_origin_xyz}" joint_origin_rpy="${joint_5_origin_rpy}" lower_limit="-${J_LIM}" upper_limit="${J_LIM}" />
-		<xacro:jaco_ring_cover suffix="3" size="small"/>
-		<xacro:jaco_joint joint_name="jaco_large_ring_cover_6_joint" type="fixed" parent="${link}_5" child="jaco_small_ring_cover_3" joint_axis_xyz="${joint_6_axis_xyz}" joint_origin_xyz="${joint_6_origin_xyz}" joint_origin_rpy="${joint_6_origin_rpy}" lower_limit="-${J_LIM}" upper_limit="${J_LIM}" />
+<!--		<xacro:jaco_ring_cover suffix="3" size="small"/>
+		<xacro:jaco_joint joint_name="jaco_large_ring_cover_6_joint" type="fixed" parent="${link}_5" child="jaco_small_ring_cover_3" joint_axis_xyz="${joint_6_axis_xyz}" joint_origin_xyz="${joint_6_origin_xyz}" joint_origin_rpy="${joint_6_origin_rpy}" lower_limit="-${J_LIM}" upper_limit="${J_LIM}" />-->
 		<xacro:jaco_link_suffix link_name="${link_finger}" suffix="1"/>
 		<xacro:jaco_finger_joint joint_name="${joint_finger_1}" type="revolute" parent="${link_hand}" child="${link_finger}_1" joint_axis_xyz="${joint_finger_1_axis_xyz}" joint_origin_xyz="${joint_finger_1_origin_xyz}" joint_origin_rpy="${joint_finger_1_origin_rpy}" lower_limit="${joint_finger_1_lower_limit}" upper_limit="${joint_finger_1_upper_limit}" />
